File: examples/demo_xe216/demo_xe216.sch (KiCad schematic (older format))
At the start: 24 parts, among them P1 CONN_02X05, P2 CONN_02X20, P3 CONN_02X20, U1 w25x40cl, U2 NC7WZ17, U3 NC7WZ17, U4 XE216-512-TQ128, Y1 25M

Commit message: linked schematics to new library names
Parts:
- C1, C2, C3, C4, C5, C6, C7, C8, C9: symbol C_Small -> Device:C_Small
- L1: symbol L_Small -> Device:L_Small
- P1: symbol CONN_02X05 -> Connector_Generic:Conn_02x05_Counter_Clockwise
- P2, P3: symbol CONN_02X20 -> Connector_Generic:Conn_02x20_Counter_Clockwise
- R1, R2, R3, R4, R5, R6: symbol R_Small -> Device:R_Small
- U1: symbol w25x40cl -> xmos_project:w25x40cl
- U2, U3: symbol NC7WZ17 -> xmos_project:NC7WZ17
- U4: symbol XE216-512-TQ128 -> xmos:XE216-512-TQ128
- Y1: symbol Crystal_Small -> Device:Crystal_Small
Connections:
- wire segments 241 -> 265
